File: hardware/TrackMAG.kicad_pcb (KiCad board)
At the start: 4 copper layers, 36 x 36 mm, 54 parts, among them J1 USB_C_Socket_USB2.0, J2 Conn_Debug, SW1 SW_RESET, SW2 SW_BOOT, U1 LSM6DS3TR-C, U2 USBLC6-2P6, U3 STM32F103C8T6, U4 LIS2MDL, U5 AMS1117-3.3, Y1 16MHz

Commit message: Center PCB
Parts:
- moved C21 96.8 mm to (131.5, 92.1)
- moved C24 96.8 mm to (147.1, 86.8)
- moved U5 96.8 mm to (147.6, 80.3)
- moved C10 96.8 mm to (134.9, 90.2)
- moved C12 96.8 mm to (146.8, 91.0)
- moved C13 96.8 mm to (143.8, 99.4)
- moved C14 96.8 mm to (134.9, 94.5)
- moved C19 96.8 mm to (154.3, 86.3)
- moved C23 96.8 mm to (155.8, 103.3)
- moved C25 96.8 mm to (141.1, 84.3)
- moved C6 96.8 mm to (154.3, 101.3)
- moved C8 96.8 mm to (154.5, 99.6)
- moved FB1 96.8 mm to (136.3, 99.4)
- moved FB2 96.8 mm to (151.0, 86.8)
- moved H3 96.8 mm to (157.5, 108.0)
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
Commit message: Add calibrate switch
Parts:
- added C23: 100n, TrackMAG:C_0402_1005Metric, F.Cu at (133.7, 95.0)
- added R12: 10k, TrackMAG:R_0402_1005Metric, F.Cu at (129.1, 104.5)
- added SW3: SW_CALIBRATE, TrackMAG:SW_Push_1P1T_XKB_TS-1187A_CALIBRATE, F.Cu at (129.8, 99.4)
- renumbered C23 to C24, C24 to C25, C25 to C26, R11 to R10, R12 to R11, R10 to R9
Connections:
- U3 pad 11: unconnected-(U3-PA1-Pad11) -> CALIBRATE
Routing:
- net CALIBRATE: track 0.00 -> 19.1 mm, vias 0 -> 4
- net GND: track 110.1 -> 104.1 mm, vias 45 -> 50

Commit message: Fix various problems, cleanup after review
Parts:
- moved C6 9.00 mm to (146.5, 96.8), turned to 180 degrees
- moved R10 6.33 mm to (149.4, 102.3), turned to 0 degrees
- moved R11 6.03 mm to (149.4, 101.2), turned to 0 degrees
- moved C4 5.94 mm to (150.7, 97.4), turned to 0 degrees
- moved C1 5.93 mm to (147.7, 94.5)
- moved C2 5.93 mm to (146.6, 94.5)
- moved C3 5.93 mm to (145.4, 94.5)
- moved C13 5.44 mm to (140.1, 95.4)
- moved C14 5.44 mm to (131.2, 90.5)
- moved C17 5.44 mm to (129.9, 84.3)
- moved C19 5.44 mm to (150.6, 82.3)
- moved C20 5.44 mm to (149.2, 82.3)
- moved C21 5.44 mm to (127.8, 88.1)
- moved C24 5.44 mm to (152.1, 99.3)
- moved C25 5.44 mm to (143.4, 82.8)
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Connections:
- J1 pad A6: /US_D+ -> /U_D+
- J1 pad A7: /US_D- -> /U_D-
- J1 pad B6: /US_D+ -> /U_D+
- J1 pad B7: /US_D- -> /U_D-
- U2 pad 1: /USB_D- -> /U_D-
- U2 pad 3: /US_D- -> /U_D+
- U2 pad 4: /US_D+ -> /USB_D+
- U2 pad 6: /USB_D+ -> /USB_D-
Routing:
- net +3.3V: track 195.1 -> 186.9 mm, vias 16 -> 14
- net +5V: track 5.53 -> 12.0 mm
- net /US_D+: track 5.12 -> 0.00 mm
- net /U_D+: track 0.00 -> 4.68 mm
- net /US_D-: track 4.27 -> 0.00 mm
- net /U_D-: track 0.00 -> 3.83 mm
- net GND: track 104.1 -> 101.5 mm, vias 50 -> 45
- net I2C_SDX: track 7.66 -> 9.79 mm
- net DRDY: track 30.8 -> 29.7 mm
- net RESET: track 65.7 -> 66.4 mm
- net SWO: track 16.4 -> 17.0 mm
- added copper zone on In1.Cu, net GND
- added copper zone on In2.Cu, net GND
